File: pcb/Mixa.sch (EAGLE design)
At the start: 51 parts

Commit message: Added BOM and Mouser PartNr
Parts:
- ATT_1: MOUSER (none) -> 688-RK09L12D0A1W
- C1: MOUSER (none) -> 710-885012206071
- C3: MOUSER (none) -> 810-C3225X7R1C226M
- C5: MOUSER (none) -> 710-885012206077
- D2: MOUSER (none) -> 621-B130-F
- JP1: MOUSER (none) -> 855-M20-8750542
- OPAMP_IS: MOUSER (none) -> 595-TL074IDR
- R14: MOUSER (none) -> 667-ERJ-3RBD2202V
- R17: MOUSER (none) -> 710-885012109014
- R18: MOUSER (none) -> 667-ERJ-3RBD104V
